File: kicad/rpi-cm5io-Kicad/CM5IO.kicad_pcb (KiCad board)
At the start: 4 copper layers, 160 x 90 mm, 87 parts, among them J1 USB3_A, J11 USB_C_Receptacle_USB2.0, J19 Barrel_Jack, J2 Conn_02x07_Odd_Even, J22 690-019-298-412, J3 USB3_A, J4 Bus_M.2_Socket_M, J5 Conn_01x22_Female, J6 USB_C_Receptacle_USB2.0_14P, J7 Micro_SD_Card_Det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

Commit message: pre final
Parts:
- removed the H6 at (211.5, 83.0)
- added ?: , , F.Cu at (211.1, 95.4)
- added ?: , , F.Cu at (210.0, 135.0)
- added H6: MountingHole, CM5IO:MountingHole_2.7mm_M2.5_DIN965, F.Cu at (84.9, 97.5)
- added H6: MountingHole, CM5IO:MountingHole_2.7mm_M2.5_DIN965, F.Cu at (85.0, 90.0)
- moved U4 7.52 mm to (210.8, 126.7)
- moved L6 1.70 mm to (90.1, 152.5)
