File: kicad/rpi-cm5io-Kicad/CM5IO.kicad_sch (KiCad schematic)
At the start: 90 parts, among them J1 USB3_A, J11 USB_C_Receptacle_USB2.0, J19 Barrel_Jack, J2 Conn_02x07_Odd_Even, J22 690-019-298-412, J3 USB3_A, J4 Bus_M.2_Socket_M, J5 Conn_01x22_Female, J6 USB_C_Receptacle_USB2.0_14P, J7 Micro_SD_Card_Det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

Commit message: pre final
Parts:
- removed C16, C17: 10u, Capacitor_SMD:C_0805_2012Metric, symbol Device:C
- U7: value ASEK-32.768KHZ-L-R-T -> 32.768KHZ
Connections:
- net M2_3v3: now also J4.68 (SUSCLK), U7.3 (Out)
Other:
- note added: "Audio in/out"
- note added: "Boot mode"
- note added: "DC-DC power"
- note added: "GPS"
- note added: "HDMI"
- note added: "M2"
- note added: "Power in"
- note added: "Rasberry Pi Computer Modele 5"
- note added: "Type C data"
- note added: "USB3"
- note removed: "5v @ 3A PSU"
- company: Copyright © 2024 Raspberry Pi Ltd. -> КПІ, ПБФ
- title: Compute Module 5 IO Board - Top Level -> title
- moved on the sheet: BT1, C1, C10, C11, C12, C13, C14, C18, C19, C20, C21, C34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
